Commit message: modifications to make z1 work in locosim
removed joint friction that was 1.0

File: robots/z1.srdf.xacro (robot description, xacro)
@@ -3,6 +3,6 @@
      <group_state name="home" group="all_legs">
 		    <joint name="joint1" value="0." />
-                    <joint name="joint2" value="0.0" />
-                    <joint name="joint3" value="0.0" />
+                    <joint name="joint2" value="0.5" />
+                    <joint name="joint3" value="-1" />
                     <joint name="joint4" value="0.0" />
                     <joint name="joint5" value="0.0" />

File: robots/z1.urdf.xacro (robot description, xacro)
@@ -1,5 +1,6 @@
 <?xml version="1.0"?>
 <robot name="z1_description" xmlns:xacro="http://www.ros.org/wiki/xacro">
-<xacro:include filename="$(find z1_description)/xacro/z1_arm.xacro"/>
+<xacro:include filename="$(find z1_description)/urdfs/z1_arm.xacro"/>
+<xacro:arg name="task_period" default="0.001" />
 <link name="world"/>
 <xacro:z1_arm parent="world">

File: urdfs/const.xacro (robot description, xacro)
@@ -103,6 +103,6 @@
     <xacro:property name="GripperMover_Izz" value="0.00035728"/>
     <!-- joint limits -->
-    <xacro:property name="jointDamping" value="1.0"/>
-    <xacro:property name="jointFriction" value="1.0"/>
+    <xacro:property name="jointDamping" value="0.0"/>
+    <xacro:property name="jointFriction" value="0.0"/>
     <xacro:property name="torqueMax" value="30.0"/>
     <xacro:property name="velocityMax" value="3.1415"/>

File: urdfs/z1_arm.xacro (robot description, xacro)
@@ -1,8 +1,11 @@
 <?xml version="1.0"?>
 <robot xmlns:xacro="http://ros.org/wiki/xacro">
+<xacro:arg name="task_period" default="0.001" />
 <xacro:macro name="z1_arm" params="parent *origin" >
-    <xacro:include filename="$(find z1_description)/xacro/const.xacro"/>
-    <xacro:include filename="$(find z1_description)/xacro/gazebo.xacro"/>
-    <xacro:include filename="$(find z1_description)/xacro/transmission.xacro"/>
+    <xacro:include filename="$(find z1_description)/urdfs/const.xacro"/>
+    <xacro:include filename="$(find z1_description)/gazebo/gazebo.urdf.xacro">
+        <xacro:arg name="task_period" value="$(arg task_period)"/>
+    </xacro:include>
+    <xacro:include filename="$(find z1_description)/urdfs/transmission.xacro"/>
     <xacro:arg name="UnitreeGripper" default="false"/>
     <joint name="base_static_joint" type="fixed">
@@ -281,4 +284,12 @@
         </gazebo>
     </xacro:if>
+    <xacro:unless value="$(arg UnitreeGripper)">
+      <joint name="ee_fixed_joint" type="fixed">
+            <origin rpy="0 0 0" xyz="0.051 0.0 0.0"/>
+            <parent link="link06"/>
+            <child link="tool0"/>
+        </joint>
+        <link name="tool0"/>
+    </xacro:unless>
     <xacro:motorTransmission name="1"/>
     <xacro:motorTransmission name="2"/>
